File: microSD.kicad_pcb (KiCad board)
At the start: 2 copper layers, 32 x 25.4 mm, 9 parts, among them IC1 74HC4050D, IC2 LP2985A, J1 microSD

Commit message: changed pin header orientation
Parts:
- J2: moved to B.Cu
- turned J2 to 0 degrees
Changed lines of the file:
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@@
 			)
 		)
-		(property "Footprint" ""
+		(property "Footprint" "Package_TO_SOT_SMD:SOT-23-5"
 			(at 0 0 180)
 			(unlocked yes)
@@
 			)
 		)
-		(property "Footprint" ""
+		(property "Footprint" "external_footprints:GCT_MEM2061-01-188-00-A_REVA"
 			(at 0 0 -90)
 			(unlocked yes)
@@
 			)
 		)
-		(property "Footprint" ""
+		(property "Footprint" "Capacitor_SMD:C_0805_2012Metric"
 			(at 0 0 180)
 			(unlocked yes)
@@
 			)
 		)
-		(property "Footprint" ""
+		(property "Footprint" "Resistor_SMD:R_0805_2012Metric"
 			(at 0 0 180)
 			(unlocked yes)
@@
 			)
 		)
-		(property "Footprint" ""
+		(property "Footprint" "LED_SMD:LED_0805_2012Metric"
 			(at 0 0 180)
 			(unlocked yes)
@@
 			)
 		)
-		(property "Footprint" ""
+		(property "Footprint" "Capacitor_SMD:C_0805_2012Metric"
 			(at 0 0 0)
 			(unlocked yes)
@@
 			)
 		)
-		(property "Footprint" ""
+		(property "Footprint" "Package_SO:SOIC-16_3.9x9.9mm_P1.27mm"
 			(at 0 0 0)
 			(unlocked yes)
@@
 	)
 	(footprint "Connector_PinHeader_2.54mm:PinHeader_1x08_P2.54mm_Vertical"
-		(layer "F.Cu")
-		(at 162.85 113.98 180)
+		(layer "B.Cu")
+		(at 162.85 113.98)
 		(descr "Through hole straight pin header, 1x08, 2.54mm pitch, single row")
 		(tags "Through hole pin header THT 1x08 2.54mm single row")
 		(property "Reference" "J2"
-			(at 0 -2.33 180)
-			(layer "F.SilkS")
+			(at 0 2.33 360)
+			(layer "B.SilkS")
 			(hide yes)
 			(effects
@@
 					(thickness 0.15)
 				)
+				(justify mirror)
 			)
 		)
 		(property "Value" "~"
-			(at 0 20.11 180)
-			(layer "F.Fab")
+			(at 0 -20.11 360)
+			(layer "B.Fab")
 			(effects
 				(font
@@
 					(thickness 0.15)
 				)
+				(justify mirror)
 			)
 		)
-		(property "Footprint" ""
+		(property "Footprint" "Connector_PinHeader_2.54mm:PinHeader_1x08_P2.54mm_Vertical"
 			(at 0 0 180)
 			(unlocked yes)
-			(layer "F.Fab")
+			(layer "B.Fab")
 			(hide yes)
 			(effects
@@
 					(size 1.27 1.27)
 				)
+				(justify mirror)
 			)
 		)
@@
 			(at 0 0 180)
 			(unlocked yes)
-			(layer "F.Fab")
+			(layer "B.Fab")
 			(hide yes)
 			(effects
@@
 					(size 1.27 1.27)
 				)
+				(justify mirror)
 			)
 		)
@@
 			(at 0 0 180)
 			(unlocked yes)
-			(layer "F.Fab")
+			(layer "B.Fab")
 			(hide yes)
 			(effects
@@
 					(size 1.27 1.27)
 				)
+				(justify mirror)
 			)
 		)
@@
 			(at 0 0 180)
 			(unlocked yes)
-			(layer "F.Fab")
+			(layer "B.Fab")
 			(hide yes)
 			(effects
@@
 					(thickness 0.15)
 				)
+				(justify mirror)
 			)
 		)
@@
 			(at 0 0 180)
 			(unlocked yes)
-			(layer "F.Fab")
+			(layer "B.Fab")
 			(hide yes)
 			(effects
@@
 					(thickness 0.15)
 				)
+				(justify mirror)
 			)
 		)
@@
 			(at 0 0 180)
 			(unlocked yes)
-			(layer "F.Fab")
+			(layer "B.Fab")
 			(hide yes)
 			(effects
@@
 					(thickness 0.15)
 				)
+				(justify mirror)
 			)
 		)
@@
 			(at 0 0 180)
 			(unlocked yes)
-			(layer "F.Fab")
+			(layer "B.Fab")
 			(hide yes)
 			(effects
@@
 					(thickness 0.15)
 				)
+				(justify mirror)
 			)
 		)
@@
 			(at 0 0 180)
 			(unlocked yes)
-			(layer "F.Fab")
+			(layer "B.Fab")
 			(hide yes)
 			(effects
@@
 					(thickness 0.15)
 				)
+				(justify mirror)
 			)
 		)
@@
 		(attr through_hole)
 		(fp_line
-			(start 1.33 1.27)
-			(end 1.33 19.11)
+			(start -1.33 -19.11)
+			(end -1.33 -1.27)
 			(stroke
 				(width 0.12)
 				(type solid)
 			)
-			(layer "F.SilkS")
+			(layer "B.SilkS")
 		)
 		(fp_line
-			(start -1.33 19.11)
-			(end 1.33 19.11)
+			(start -1.33 1.33)
+			(end -1.33 0)
 			(stroke
 				(width 0.12)
 				(type solid)
 			)
-			(layer "F.SilkS")
+			(layer "B.SilkS")
 		)
 		(fp_line
-			(start -1.33 1.27)
-			(end 1.33 1.27)
+			(start 0 1.33)
+			(end -1.33 1.33)
 			(stroke
 				(width 0.12)
 				(type solid)
 			)
-			(layer "F.SilkS")
+			(layer "B.SilkS")
 		)
 		(fp_line
-			(start -1.33 1.27)
-			(end -1.33 19.11)
+			(start 1.33 -19.11)
+			(end -1.33 -19.11)
 			(stroke
 				(width 0.12)
 				(type solid)
 			)
-			(layer "F.SilkS")
+			(layer "B.SilkS")
 		)
 		(fp_line
-			(start -1.33 0)
-			(end -1.33 -1.33)
+			(start 1.33 -19.11)
+			(end 1.33 -1.27)
 			(stroke
 				(width 0.12)
 				(type solid)
 			)
-			(layer "F.SilkS")
+			(layer "B.SilkS")
 		)
 		(fp_line
-			(start -1.33 -1.33)
-			(end 0 -1.33)
+			(start 1.33 -1.27)
+			(end -1.33 -1.27)
 			(stroke
 				(width 0.12)
 				(type solid)
 			)
-			(layer "F.SilkS")
+			(layer "B.SilkS")
 		)
 		(fp_line
-			(start 1.8 19.55)
-			(end 1.8 -1.8)
+			(start -1.8 -19.55)
+			(end -1.8 1.8)
 			(stroke
 				(width 0.05)
 				(type solid)
 			)
-			(layer "F.CrtYd")
+			(layer "B.CrtYd")
 		)
 		(fp_line
-			(start 1.8 -1.8)
-			(end -1.8 -1.8)
+			(start -1.8 1.8)
+			(end 1.8 1.8)
 			(stroke
 				(width 0.05)
 				(type solid)
 			)
-			(layer "F.CrtYd")
+			(layer "B.CrtYd")
 		)
 		(fp_line
-			(start -1.8 19.55)
-			(end 1.8 19.55)
+			(start 1.8 -19.55)
+			(end -1.8 -19.55)
 			(stroke
 				(width 0.05)
 				(type solid)
 			)
-			(layer "F.CrtYd")
+			(layer "B.CrtYd")
 		)
 		(fp_line
-			(start -1.8 -1.8)
-			(end -1.8 19.55)
+			(start 1.8 1.8)
+			(end 1.8 -19.55)
 			(stroke
 				(width 0.05)
 				(type solid)
 			)
-			(layer "F.CrtYd")
+			(layer "B.CrtYd")
 		)
 		(fp_line
-			(start 1.27 19.05)
-			(end -1.27 19.05)
+			(start -1.27 -19.05)
+			(end 1.27 -19.05)
 			(stroke
 				(width 0.1)
 				(type solid)
 			)
-			(layer "F.Fab")
+			(layer "B.Fab")
 		)
 		(fp_line
-			(start 1.27 -1.27)
-			(end 1.27 19.05)
+			(start -1.27 0.635)
+			(end -1.27 -19.05)
 			(stroke
 				(width 0.1)
 				(type solid)
 			)
-			(layer "F.Fab")
+			(layer "B.Fab")
 		)
 		(fp_line
-			(start -0.635 -1.27)
-			(end 1.27 -1.27)
+			(start -0.635 1.27)
+			(end -1.27 0.635)
 			(stroke
 				(width 0.1)
 				(type solid)
 			)
-			(layer "F.Fab")
+			(layer "B.Fab")
 		)
 		(fp_line
-			(start -1.27 19.05)
-			(end -1.27 -0.635)
+			(start 1.27 -19.05)
+			(end 1.27 1.27)
 			(stroke
 				(width 0.1)
 				(type solid)
 			)
-			(layer "F.Fab")
+			(layer "B.Fab")
 		)
 		(fp_line
-			(start -1.27 -0.635)
-			(end -0.635 -1.27)
+			(start 1.27 1.27)
+			(end -0.635 1.27)
 			(stroke
 				(width 0.1)
 				(type solid)
 			)
-			(layer "F.Fab")
+			(layer "B.Fab")
 		)
 		(fp_text user "${REFERENCE}"
-			(at 0 8.89 -90)
-			(layer "F.Fab")
+			(at 0 -8.89 90)
+			(layer "B.Fab")
 			(effects
 				(font
@@
 					(thickness 0.15)
 				)
+				(justify mirror)
 			)
 		)
 		(pad "1" thru_hole rect
-			(at 0 0 180)
+			(at 0 0)
 			(size 1.7 1.7)
 			(drill 1)
@@
 		)
 		(pad "2" thru_hole oval
-			(at 0 2.54 180)
+			(at 0 -2.54)
 			(size 1.7 1.7)
 			(drill 1)
@@
 		)
 		(pad "3" thru_hole oval
-			(at 0 5.08 180)
+			(at 0 -5.08)
 			(size 1.7 1.7)
 			(drill 1)
@@
 		)
 		(pad "4" thru_hole oval
-			(at 0 7.62 180)
+			(at 0 -7.62)
 			(size 1.7 1.7)
 			(drill 1)
@@
 		)
 		(pad "5" thru_hole oval
-			(at 0 10.16 180)
+			(at 0 -10.16)
 			(size 1.7 1.7)
 			(drill 1)
@@
 		)
 		(pad "6" thru_hole oval
-			(at 0 12.7 180)
+			(at 0 -12.7)
 			(size 1.7 1.7)
 			(drill 1)
@@
 		)
 		(pad "7" thru_hole oval
-			(at 0 15.24 180)
+			(at 0 -15.24)
 			(size 1.7 1.7)
 			(drill 1)
@@
 		)
 		(pad "8" thru_hole oval
-			(at 0 17.78 180)
+			(at 0 -17.78)
 			(size 1.7 1.7)
 			(drill 1)
@@
 		(model "${KICAD8_3DMODEL_DIR}/Connector_PinHeader_2.54mm.3dshapes/PinHeader_1x08_P2.54mm_Vertical.wrl"
 			(offset
-				(xyz 0 0 -1.5)
+				(xyz 0 0 0)
 			)
 			(scale
@@
 			)
 			(rotate
-				(xyz 0 180 0)
+				(xyz 0 0 0)
 			)
 		)

Commit message: external STEP folder rename
Parts:
- J1: footprint external_footprints:GCT_MEM2061-01-188-00-A_REVA -> external_footprints:MEM2061-01-188-00-A
Changed lines of the file:
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@@
 		)
 	)
-	(footprint "external_footprints:GCT_MEM2061-01-188-00-A_REVA"
+	(footprint "external_footprints:MEM2061-01-188-00-A"
 		(layer "F.Cu")
 		(at 140.825 105.125 -90)
@@
 			)
 		)
-		(property "Footprint" "external_footprints:GCT_MEM2061-01-188-00-A_REVA"
+		(property "Footprint" "external_footprints:MEM2061-01-188-00-A"
 			(at 0 0 -90)
 			(unlocked yes)
@@
 			)
 		)
-		(model "${KIPRJMOD}/external/STEP/MEM2061-01-188-00-A_REVA.step"
+		(model "${KIPRJMOD}/external/3dmodels/MEM2061-01-188-00-A.step"
 			(offset
 				(xyz 0 0 0)
@@
 		(tags "Through hole pin header THT 1x08 2.54mm single row")
 		(property "Reference" "J2"
-			(at 0 2.33 360)
+			(at 0 2.33 0)
 			(layer "B.SilkS")
 			(hide yes)
@@
 		)
 		(property "Value" "~"
-			(at 0 -20.11 360)
+			(at 0 -20.11 0)
 			(layer "B.Fab")
 			(effects
