File: microSD.kicad_sch (KiCad schematic)
At the start: 8 parts, among them IC1 74HC4050D, IC2 LP2985A, J1 microSD

Commit message: build!: upgrade schematic and board to KiCad 10
Parts:
- J2: value ~ -> (none)
