File: microSD.kicad_sch (KiCad schematic)
At the start: 8 parts, among them IC1 74HC4050D, IC2 LP2985A, J1 microSD

Commit message: docs: fill in the title block
Other:
- company: (none) -> UHasselt, Solar Cooker
Changed lines of the file:
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@@
 	(title_block
 		(title "microSD")
-		(date "2024-03-06")
+		(date "2026-10-18")
+		(rev "1.0")
+		(company "UHasselt, Solar Cooker")
+		(comment 1 "Based on the Adafruit MicroSD card breakout board+")
+		(comment 2 "Design: Lowie Van Vyve")
+		(comment 3 "github.com/solar-cooker-UHasselt/kicad-adafruit-microsd")
 	)
 	(junction
